Commit message: Add joint_state_publisher for the caster wheels so they appear at RViZ

File: urdf/mobile_manipulator.gazebo.xacro (robot description, xacro)
@@ -81,9 +81,21 @@
   <gazebo>
       <plugin name="gazebo_ros_control" filename="libgazebo_ros_control.so">
-      <robotNamespace>/</robotNamespace>
-      <controlPeriod>0.001</controlPeriod>
-      <legacyModeNS>false</legacyModeNS>
-      <robotSimType>gazebo_ros_control/DefaultRobotHWSim</robotSimType>
+        <robotNamespace>/</robotNamespace>
+        <controlPeriod>0.001</controlPeriod>
+        <legacyModeNS>false</legacyModeNS>
+        <robotSimType>gazebo_ros_control/DefaultRobotHWSim</robotSimType>
       </plugin>
   </gazebo>
+  <gazebo>
+    <plugin name="joint_state_publisher" filename="libgazebo_ros_joint_state_publisher.so">
+      <jointName>
+                  MiR__base_fl_caster_rotation_joint, MiR__base_fl_caster_wheel_joint,
+                  MiR__base_bl_caster_rotation_joint, MiR__base_bl_caster_wheel_joint,
+                  MiR__base_fr_caster_rotation_joint, MiR__base_fr_caster_wheel_joint,
+                  MiR__base_br_caster_rotation_joint, MiR__base_br_caster_wheel_joint
+      </jointName>
+      <updateRate>100.0</updateRate>
+      <alwaysOn>true</alwaysOn>
+    </plugin>
+  </gazebo>
 </robot>

File: urdf/mobile_manipulator.urdf.xacro (robot description, xacro)
@@ -9,4 +9,73 @@
 <!-- ################# Properties ################ -->
 <!-- ############################################# -->
+  <!-- ############### MiR ############ -->
+  <!-- ################################ -->
+    <xacro:property name="deg_to_rad" value="0.017453293" />
+    <xacro:property name="mir_100_base_mass" value="58.0" />
+    <xacro:property name="mir_100_act_wheel_radius" value="0.0625" />
+    <xacro:property name="mir_100_act_wheel_width" value="0.032" />
+    <xacro:property name="mir_100_act_wheel_mass" value="1.0" />
+    <xacro:property name="mir_100_act_wheel_dx" value="0.037646" />
+    <xacro:property name="mir_100_act_wheel_dy" value="0.222604" />
+    <xacro:property name="mir_100_caster_wheel_radius" value="${mir_100_act_wheel_radius}" />
+    <xacro:property name="mir_100_caster_wheel_width" value="${mir_100_act_wheel_width}" />
+    <xacro:property name="mir_100_caster_wheel_mass" value="${mir_100_act_wheel_mass}" />
+    <xacro:property name="mir_100_caster_wheel_dx" value="-0.0382" />
+    <xacro:property name="mir_100_caster_wheel_dy" value="0" />
+    <xacro:property name="mir_100_caster_wheel_dz" value="-0.094" />
+    <xacro:property name="mir_100_front_caster_wheel_base_dx" value="0.341346" />
+    <xacro:property name="mir_100_back_caster_wheel_base_dx" value="-0.270154" />
+    <xacro:property name="mir_100_caster_wheel_base_dy" value="0.203" />
+    <xacro:property name="mir_100_caster_wheel_base_dz" value="${mir_100_caster_wheel_radius-mir_100_caster_wheel_dz}" />
+    <xacro:property name="imu_stdev" value="0.00017" />
+    <xacro:property name="imu_update_rate" value="50" />
+  <!-- ################################ -->
+  <!-- ############### MiR ############ -->
+  <!-- ############### UR10 ############ -->
+  <!-- ################################ -->
+    <!-- Inertia parameters -->
+      <xacro:property name="ur10_base_mass" value="4.0" />  <!-- This mass might be incorrect -->
+      <xacro:property name="ur10_shoulder_mass" value="7.778" />
+      <xacro:property name="ur10_upper_arm_mass" value="12.93" />
+      <xacro:property name="ur10_forearm_mass" value="3.87" />
+      <xacro:property name="ur10_wrist_1_mass" value="1.96" />
+      <xacro:property name="ur10_wrist_2_mass" value="1.96" />
+      <xacro:property name="ur10_wrist_3_mass" value="0.202" />
+    <!-- Kinematic model -->
+    <!-- Properties from urcontrol.conf -->
+      <xacro:property name="d1" value="0.1273" />
+      <xacro:property name="a2" value="-0.612" />
+      <xacro:property name="a3" value="-0.5723" />
+      <xacro:property name="d4" value="0.163941" />
+      <xacro:property name="d5" value="0.1157" />
+      <xacro:property name="d6" value="0.0922" />
+    <!-- link lengths used in model -->
+      <xacro:property name="ur10_shoulder_height" value="${d1}" />
+      <xacro:property name="ur10_upper_arm_length" value="${-a2}" />
+      <xacro:property name="ur10_forearm_length" value="${-a3}" />
+      <xacro:property name="ur10_wrist_1_length" value="${d4 - ur10_elbow_offset - ur10_shoulder_offset}" />
+      <xacro:property name="ur10_wrist_2_length" value="${d5}" />
+      <xacro:property name="ur10_wrist_3_length" value="${d6}" />
+    <!-- Arbitrary offsets for shoulder/elbow joints -->
+      <xacro:property name="ur10_shoulder_offset" value="0.220941" />  <!-- measured from model -->
+      <xacro:property name="ur10_elbow_offset" value="-0.1719" /> <!-- measured from model -->
+      <xacro:property name="ur10_upper_arm_inertia_offset" value="0.045" />  <!-- measured from model -->
+    <xacro:property name="ur10_shoulder_pan_lower_limit" value="${-pi}"/>
+    <xacro:property name="ur10_shoulder_pan_upper_limit" value="${pi}"/>
+    <xacro:property name="ur10_shoulder_lift_lower_limit" value="${-pi}"/>
+    <xacro:property name="ur10_shoulder_lift_upper_limit" value="${pi}"/>
+    <xacro:property name="ur10_elbow_joint_lower_limit" value="${-pi}"/>
+    <xacro:property name="ur10_elbow_joint_upper_limit" value="${pi}"/>
+    <xacro:property name="ur10_wrist_1_lower_limit" value="${-pi}"/>
+    <xacro:property name="ur10_wrist_1_upper_limit" value="${pi}"/>
+    <xacro:property name="ur10_wrist_2_lower_limit" value="${-pi}"/>
+    <xacro:property name="ur10_wrist_2_upper_limit" value="${pi}"/>
+    <xacro:property name="ur10_wrist_3_lower_limit" value="${-pi}"/>
+    <xacro:property name="ur10_wrist_3_upper_limit" value="${pi}"/>
+    <xacro:property name="ur10_safety_limits" value="false"/>
+    <xacro:property name="ur10_safety_pos_margin" value="0.15"/>
+    <xacro:property name="ur10_safety_k_position" value="20"/>
+  <!-- ################################ -->
+  <!-- ############### UR10 ############ -->
   <!-- ######## Barrett Hand ########## -->
   <!-- ################################ -->
@@ -20,4 +89,464 @@
 <!-- ############################################# -->
 <!-- ################# Properties ################ -->
+<!-- ################# Macros ################ -->
+<!-- ######################################### -->
+  <!-- ############### MiR ############ -->
+  <!-- ################################ -->
+    <xacro:macro name="actuated_wheel" params="locationprefix locationright">
+      <joint name="MiR__base_${locationprefix}_wheel_joint" type="continuous">
+        <origin xyz="0.0 ${-mir_100_act_wheel_dy * locationright} ${mir_100_act_wheel_radius}" rpy="0 0 0" />
+        <parent link="MiR_base_link" />
+        <child link="MiR_${locationprefix}_wheel_link" />
+        <axis xyz="0 1 0" />
+        <limit effort="100" velocity="20.0" />
+      </joint>
+      <link name="MiR_${locationprefix}_wheel_link">
+        <xacro:cylinder_inertial mass="${mir_100_act_wheel_mass}" radius="${mir_100_act_wheel_radius}" length="${mir_100_act_wheel_width}">
+        <origin xyz="0 0 0" rpy="${0.5 * pi} 0 0" />
+        </xacro:cylinder_inertial>
+        <visual>
+          <origin xyz="0 0 0" rpy="0 0 0" />
+          <geometry>
+            <mesh filename="package://mobile_manipulator/mesh/mir100/visual/wheel.stl" />
+          </geometry>
+          <xacro:insert_block name="material_dark_grey" />
+        </visual>
+        <collision>
+          <origin xyz="0 0 0" rpy="0 0 0" />
+          <geometry>
+            <mesh filename="package://mobile_manipulator/mesh/mir100/visual/wheel.stl" />
+          </geometry>
+        </collision>
+      </link>
+      <gazebo reference="MiR_${locationprefix}_wheel_link">
+        <material>Gazebo/DarkGrey</material>
+      </gazebo>
+    </xacro:macro>
+    <xacro:macro name="caster_wheel" params="locationprefix locationright wheel_base_dx">
+      <!-- caster hub -->
+        <joint name="MiR__base_${locationprefix}_caster_rotation_joint" type="continuous">
+          <origin xyz="${wheel_base_dx} ${-mir_100_caster_wheel_base_dy * locationright} ${mir_100_caster_wheel_base_dz}" rpy="0 0 0" />
+          <parent link="MiR_base_link" />
+          <child link="MiR_${locationprefix}_caster_rotation_link" />
+          <axis xyz="0 0 1" />
+          <dynamics damping="0.01" friction="0.0"/>
+        </joint>
+        <link name="MiR_${locationprefix}_caster_rotation_link">
+          <inertial>
+            <!-- <origin xyz="0 0 -0.042500000044" rpy="${0.5 * pi} ${24 * deg_to_rad} ${1.5 * pi}" /> -->
+            <origin xyz="0 0 -0.042500000044" rpy="${24 * deg_to_rad} 0 ${0.5 * pi} " />
+            <mass value="0.3097539019" />
+            <inertia
+              ixx="0.0005844517978"
+              ixy="0"
+              ixz="0"
+              iyy="0.00052872551237"
+              iyz="0"
+              izz="0.00017923555074" />
+          </inertial>
+          <visual>
+            <origin xyz="0 0 0" rpy="0 0 0" />
+            <geometry>
+              <mesh filename="package://mobile_manipulator/mesh/mir100/visual/caster_wheel_base.stl" />
+            </geometry>
+            <xacro:insert_block name="material_silver" />
+          </visual>
+          <collision>
+            <origin xyz="0 0 0" rpy="0 0 0" />
+            <geometry>
+              <mesh filename="package://mobile_manipulator/mesh/mir100/collision/caster_wheel_base.stl" />
+            </geometry>
+          </collision>
+        </link>
+        <gazebo reference="MiR_${locationprefix}_caster_rotation_link">
+          <material>Gazebo/Grey</material>
+        </gazebo>
+      <!-- caster wheel -->
+        <joint name="MiR__base_${locationprefix}_caster_wheel_joint" type="continuous">
+          <origin xyz="${mir_100_caster_wheel_dx} ${-mir_100_caster_wheel_dy * locationright} ${mir_100_caster_wheel_dz}" rpy="0 0 0" />
+          <parent link="MiR_${locationprefix}_caster_rotation_link" />
+          <child link="MiR_${locationprefix}_caster_wheel_link" />
+          <axis xyz="0 1 0" />
+        </joint>
+        <link name="MiR_${locationprefix}_caster_wheel_link">
+          <xacro:cylinder_inertial mass="${mir_100_caster_wheel_mass}" radius="${mir_100_caster_wheel_radius}" length="${mir_100_caster_wheel_width}">
+            <origin xyz="0 0 0" rpy="${0.5 * pi} 0 0" />
+          </xacro:cylinder_inertial>
+          <visual>
+            <origin xyz="0 0 0" rpy="0 0 0" />
+            <geometry>
+              <mesh filename="package://mobile_manipulator/mesh/mir100/visual/wheel.stl" />
+            </geometry>
+            <xacro:insert_block name="material_dark_grey" />
+          </visual>
+          <collision>
+            <origin xyz="0 0 0" rpy="0 0 0" />
+            <geometry>
+              <mesh filename="package://mobile_manipulator/mesh/mir100/visual/wheel.stl" />
+            </geometry>
+          </collision>
+        </link>
+        <gazebo reference="MiR_${locationprefix}_caster_wheel_link">
+          <material>Gazebo/DarkGrey</material>
+        </gazebo>
+    </xacro:macro>
+  <!-- ################################ -->
+  <!-- ############### MiR ############ -->
+<!-- ######################################### -->
+<!-- ################# Macros ################ -->
+<!-- #################### MiR #################### -->
+<!-- ############################################# -->
+  <link name="MiR_footprint" />
+  <joint name="MiR__footprint_to_base_joint" type="fixed">
+    <parent link="MiR_footprint" />
+    <child link="MiR_base_link" />
+    <origin xyz="0 0 0" rpy="0 0 0" />
+  </joint>
+  <link name="MiR_base_link">
+    <xacro:box_inertial mass="${mir_100_base_mass}" x="0.9" y="0.58" z="0.3">
+      <origin xyz="${mir_100_act_wheel_dx} 0 0.20" rpy="0 0 0" />
+    </xacro:box_inertial>
+    <visual>
+      <origin xyz="${mir_100_act_wheel_dx} 0 0" rpy="0 0 0" />
+      <geometry>
+        <mesh filename="package://mobile_manipulator/mesh/mir100/visual/mir_100_base.stl" />
+      </geometry>
+      <xacro:insert_block name="material_white" />
+    </visual>
+    <collision>
+      <origin xyz="${mir_100_act_wheel_dx} 0 0" rpy="0 0 0" />
+      <geometry>
+        <mesh filename="package://mobile_manipulator/mesh/mir100/collision/mir_100_base.stl" />
+      </geometry>
+    </collision>
+  </link>
+  <gazebo reference="MiR_base_link">
+    <material>Gazebo/White</material>
+  </gazebo>
+    <!-- wheels -->
+      <xacro:actuated_wheel locationprefix="left" locationright="-1"/>
+      <xacro:actuated_wheel locationprefix="right" locationright="1"/>
+      <xacro:caster_wheel locationprefix="fl" locationright="-1" wheel_base_dx="${mir_100_front_caster_wheel_base_dx}"/>
+      <xacro:caster_wheel locationprefix="fr" locationright="1" wheel_base_dx="${mir_100_front_caster_wheel_base_dx}"/>
+      <xacro:caster_wheel locationprefix="bl" locationright="-1" wheel_base_dx="${mir_100_back_caster_wheel_base_dx}"/>
+      <xacro:caster_wheel locationprefix="br" locationright="1" wheel_base_dx="${mir_100_back_caster_wheel_base_dx}"/>
+      <xacro:MiR_wheel_transmissions/>
+      <xacro:set_all_wheel_frictions/>
+    -<xacro:p3d_base_controller/>
+    <joint name="MiR__base_to_surface_joint" type="fixed">
+      <origin xyz="${mir_100_act_wheel_dx} 0 0.352" rpy="0 0 0" />
+      <parent link="MiR_base_link" />
+      <child link="MiR_surface" />
+      <axis xyz="0 0 1" />
+    </joint>
+    <link name="MiR_surface"/>
+  <!-- IMU -->
+    <joint name="MiR__base_to_imu_joint" type="fixed">
+      <parent link="MiR_base_link" />
+      <child link="MiR_imu_link" />
+      <origin xyz="0.0 0.0 0.25" rpy="0 0 0" />  <!-- same as real MiR -->
+    </joint>
+    <link name="MiR_imu_link" />
+    <xacro:imu link="MiR_imu_link" imu_topic="Mir/imu_data" update_rate="${imu_update_rate}" stdev="${imu_stdev}" />
+    <!-- Create an alias for imu_link. This is necessary because the real MiR's
+          TF has imu_link, but the imu_data topic is published in the imu_frame
+          frame. -->
+      <joint name="MiR__imu_link_to_imu_frame_joint" type="fixed">
+        <parent link="MiR_imu_link" />
+        <child link="MiR_imu_frame" />
+        <origin xyz="0 0 0" rpy="0 0 0" />
+      </joint>
+      <link name="MiR_imu_frame" />
+  <!-- Laser scanners -->
+    <joint name="MiR__base_to_front_laser_joint" type="fixed">
+      <parent link="MiR_base_link" />
+      <child link="MiR_front_laser_link" />
+      <origin xyz="0.4288 0.2358 0.1914" rpy="0.0 0.0 ${0.25 * pi}" />  <!-- from visually matching up the meshes of the MiR and the laser scanner -->
+    </joint>
+    <xacro:sick_s300 link="MiR_front_laser_link" topic="Mir/back_lscan" />
+    <joint name="Mir__base_to_back_laser_joint" type="fixed">
+      <parent link="MiR_base_link" />
+      <child link="MiR_back_laser_link" />
+      <origin xyz="-0.3548 -0.2352 0.1914" rpy="0.0 0.0 ${-0.75 * pi}" />  <!-- from visually matching up the meshes of the MiR and the laser scanner -->
+    </joint>
+    <xacro:sick_s300 link="MiR_back_laser_link" topic="Mir/back_lscan" />
+  <!-- Ultrasound sensors -->
+    <link name="MiR_right_us_frame" />
+    <joint name="MiR__base_to_right_us_joint" type="fixed">   <!-- right ultrasound -->
+      <parent link="MiR_base_link" />
+      <child link="MiR_right_us_frame" />
+      <origin xyz="0.45 -0.12 0.16 " rpy="0 0 0" />  <!-- from visually matching to the mesh of the MiR -->
+    </joint>
+    <xacro:ultrasound_gazebo link="MiR_right_us_frame" topic="/MiR/right_ultrasound" update_rate="5"
+                                                  range_min="0.01" range_max="0.75"
+                                                  horizental_min_angle="-0.25" horizental_max_angle="0.25"
+                                                  vertical_min_angle="-0.25" vertical_max_angle="0.25"/>
+    <link name="MiR_left_us_frame" />
+    <joint name="MiR__base_to_left_us_joint" type="fixed">   <!-- right ultrasound -->
+      <parent link="MiR_base_link" />
+      <child link="MiR_left_us_frame" />
+      <origin xyz="0.45 -0.12 0.16 " rpy="0 0 0" />  <!-- from visually matching to the mesh of the MiR -->
+    </joint>
+    <xacro:ultrasound_gazebo link="MiR_left_us_frame" topic="/MiR/left_ultrasound" update_rate="10"
+                                                  range_min="0.01" range_max="0.75"
+                                                  horizental_min_angle="-0.25" horizental_max_angle="0.25"
+                                                  vertical_min_angle="-0.25" vertical_max_angle="0.25"/>
+<!-- ############################################# -->
+<!-- #################### MiR #################### -->
+<!-- #################### UR10 ################### -->
+<!-- ############################################# -->
+  <link name="UR10_base_link" >
+    <visual>
+      <geometry>
+        <mesh filename="package://mobile_manipulator/mesh/ur10/visual/base.dae"/>
+      </geometry>
+      <material name="LightGrey">
+        <color rgba="0.7 0.7 0.7 1.0"/>
+      </material>
+    </visual>
+    <collision>
+      <geometry>
+        <mesh filename="package://mobile_manipulator/mesh/ur10/collision/base.stl"/>
+      </geometry>
+    </collision>
+    <xacro:cylinder_inertial radius="0.075" length="0.038" mass="${ur10_base_mass}">
+      <origin xyz="0.0 0.0 0.0" rpy="0 0 0" />
+    </xacro:cylinder_inertial>
+  </link>
+  <gazebo reference="UR10_base_link">
+    <selfCollide>true</selfCollide>
+  </gazebo>
+  <joint name="UR10__base_to_shoulder_pan_joint" type="revolute">
+    <parent link="UR10_base_link" />
+    <child link = "UR10_shoulder_pan_link" />
+    <origin xyz="0.0 0.0 ${ur10_shoulder_height}" rpy="0.0 0.0 0.0" />
+    <axis xyz="0 0 1" />
+    <limit lower="${ur10_shoulder_pan_lower_limit}" upper="${ur10_shoulder_pan_upper_limit}" effort="330.0" velocity="2.16"/>
+    <xacro:if value="${ur10_safety_limits}">
+      <safety_controller soft_lower_limit="${ur10_shoulder_pan_lower_limit + ur10_safety_pos_margin}" soft_upper_limit="${ur10_shoulder_pan_upper_limit - ur10_safety_pos_margin}" k_position="${ur10_safety_k_position}" k_velocity="0.0"/>
+    </xacro:if>
+    <dynamics damping="0.0" friction="0.0"/>
+  </joint>
+  <link name="UR10_shoulder_pan_link">
+    <visual>
+      <geometry>
+        <mesh filename="package://mobile_manipulator/mesh/ur10/visual/shoulder.dae"/>
+      </geometry>
+      <material name="LightGrey">
+        <color rgba="0.7 0.7 0.7 1.0"/>
+      </material>
+    </visual>
+    <collision>
+      <geometry>
+        <mesh filename="package://mobile_manipulator/mesh/ur10/collision/shoulder.stl"/>
+      </geometry>
+    </collision>
+    <xacro:cylinder_inertial radius="0.075" length="0.178" mass="${ur10_shoulder_mass}">
+      <origin xyz="0.0 0.0 0.0" rpy="0 0 0" />
+    </xacro:cylinder_inertial>
+  </link>
+  <gazebo reference="UR10_shoulder_pan_link">
+    <selfCollide>true</selfCollide>
+  </gazebo>
+  <joint name="UR10__shoulder_pan_to_upper_arm_joint" type="revolute">
+    <parent link="UR10_shoulder_pan_link" />
+    <child link = "UR10_upper_arm_link" />
+    <origin xyz="0.0 ${ur10_shoulder_offset} 0.0" rpy="0.0 0.0 0.0" />
+    <axis xyz="0 1 0" />
+    <limit lower="${ur10_shoulder_lift_lower_limit}" upper="${ur10_shoulder_lift_upper_limit}" effort="330.0" velocity="2.16"/>
+    <xacro:if value="${ur10_safety_limits}">
+      <safety_controller soft_lower_limit="${ur10_shoulder_lift_lower_limit + ur10_safety_pos_margin}" soft_upper_limit="${ur10_shoulder_lift_upper_limit - ur10_safety_pos_margin}" k_position="${ur10_safety_k_position}" k_velocity="0.0"/>
+    </xacro:if>
+    <dynamics damping="0.0" friction="0.0"/>
+  </joint>
+  <link name="UR10_upper_arm_link">
+    <visual>
+      <geometry>
+        <mesh filename="package://mobile_manipulator/mesh/ur10/visual/upperarm.dae"/>
+      </geometry>
+      <material name="LightGrey">
+        <color rgba="0.7 0.7 0.7 1.0"/>
+      </material>
+    </visual>
+    <collision>
+      <geometry>
+        <mesh filename="package://mobile_manipulator/mesh/ur10/collision/upperarm.stl"/>
+      </geometry>
+    </collision>
+    <xacro:cylinder_inertial radius="0.075" length="${-a2}" mass="${ur10_upper_arm_mass}">
+      <origin xyz="0.0 ${-ur10_upper_arm_inertia_offset} ${-a2/2.0}" rpy="0 0 0" />
+    </xacro:cylinder_inertial>
+  </link>
+  <gazebo reference="UR10_upper_arm_link">
+    <selfCollide>true</selfCollide>
+  </gazebo>
+  <joint name="UR10__upper_arm_to_fore_arm_joint" type="revolute">
+    <parent link="UR10_upper_arm_link" />
+    <child link = "UR10_fore_arm_link" />
+    <origin xyz="0.0 ${ur10_elbow_offset} ${ur10_upper_arm_length}" rpy="0.0 0.0 0.0" />
+    <axis xyz="0 1 0" />
+    <limit lower="${ur10_elbow_joint_lower_limit}" upper="${ur10_elbow_joint_upper_limit}" effort="150.0" velocity="3.15"/>
+    <xacro:if value="${ur10_safety_limits}">
+      <safety_controller soft_lower_limit="${ur10_elbow_joint_lower_limit + ur10_safety_pos_margin}" soft_upper_limit="${ur10_elbow_joint_upper_limit - ur10_safety_pos_margin}" k_position="${ur10_safety_k_position}" k_velocity="0.0"/>
+    </xacro:if>
+    <dynamics damping="0.0" friction="0.0"/>
+  </joint>
+  <link name="UR10_fore_arm_link">
+    <visual>
+        <geometry>
+        <mesh filename="package://mobile_manipulator/mesh/ur10/visual/forearm.dae"/>
+      </geometry>
+      <material name="LightGrey">
+        <color rgba="0.7 0.7 0.7 1.0"/>
+      </material>
+    </visual>
+    <collision>
+      <geometry>
+        <mesh filename="package://mobile_manipulator/mesh/ur10/collision/forearm.stl"/>
+      </geometry>
+    </collision>
+    <gazebo>
+      <selfCollide>true</selfCollide>
+    </gazebo>
+    <xacro:cylinder_inertial radius="0.075" length="${-a3}" mass="${ur10_forearm_mass}">
+      <origin xyz="0.0 0.0 ${-a3/2.0}" rpy="0 0 0" />
+    </xacro:cylinder_inertial>
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
File: urdf/sensors.ultrasound.urdf.xacro (robot description, xacro)
@@ -7,5 +7,5 @@
       <gazebo reference="${link}">
         <sensor type="ray" name="sonar">
-          <pose>0.25 0 0 0 0 0</pose>
+          <pose>0 0 0 0 0 0</pose>
           <update_rate>${update_rate}</update_rate>
           <ray>
