Commit message: Using Joint Position Controllers...Before adding Effort Controller

File: urdf/bh282/bh282.urdf.xacro (robot description, xacro)
@@ -13,8 +13,9 @@
     <!-- #################################################### -->
         <xacro:macro name="BH282_hand" params="parent">
-            <joint name="BH282_base_joint" type="fixed">
+            <joint name="BH282_base_joint_fixed" type="fixed">
                 <!-- To Attach the Gripper to the Arm -->
-                <origin xyz="0 0 0" rpy="0 ${0.5 * pi} 0" />
-                <!-- <origin xyz="0 0 0" rpy="0 0 0" /> -->
+                <!-- Change This if you would like to run the gripper stand-alone -->
+                <!-- <origin xyz="0 0 0" rpy="0 ${0.5 * pi} 0" /> -->
+                <origin xyz="0 0 0" rpy="0 0 0" />
                 <parent link="${parent}"/>
                 <child link="BH282_base_link"/>
@@ -231,5 +232,5 @@
                     </collision>
                 </link>
-                <joint name="BH282__base_to_finger_31_joint" type="fixed">
+                <joint name="BH282__base_to_finger_31_joint_fixed" type="fixed">
                     <parent link="BH282_base_link"/>
                     <child link="BH282_finger_31_link"/>

File: urdf/mir100/mir100.gazebo.xacro (robot description, xacro)
@@ -61,5 +61,5 @@
                     <wheelDiameter>${2*wheel_radius}</wheelDiameter>
                     <wheelTorque>10</wheelTorque>
-                    <publishTf>1</publishTf>
+                    <publishTf>false</publishTf>
                     <odometryFrame>map</odometryFrame>
                     <commandTopic>MiR/controller/cmd_vel</commandTopic>

File: urdf/mir100/mir100.urdf.xacro (robot description, xacro)
@@ -22,4 +22,6 @@
         <xacro:property name="imu_stdev" value="0.00017" />
         <xacro:property name="imu_update_rate" value="50" />
+        <xacro:property name="wheel_separation" value="0.445208" />
+        <xacro:property name="wheel_radius" value="0.0625" />
     <!-- ############################################# -->
     <!-- ################# Properties ################ -->
@@ -116,5 +118,5 @@
         </xacro:macro>
         <xacro:macro name="MiR100_mobile_robot" params="parent">
-            <joint name="MiR__base_joint" type="fixed">
+            <joint name="MiR__base_joint_fixed" type="fixed">
                 <parent link="${parent}" />
                 <child link="MiR_base_link" />
@@ -149,5 +151,5 @@
             <xacro:caster_hub locationprefix="br" locationright="1" wheel_base_dx="${mir_100_back_caster_wheel_base_dx}"/>
             <xacro:caster_wheel locationprefix="br" locationright="1" wheel_base_dx="${mir_100_back_caster_wheel_base_dx}"/>
-            <joint name="MiR__base_to_surface_joint" type="fixed">
+            <joint name="MiR__base_to_surface_joint_fixed" type="fixed">
                 <origin xyz="${mir_100_act_wheel_dx} 0 0.352" rpy="0 0 0" />
                 <parent link="MiR_base_link" />
@@ -157,5 +159,5 @@
             <link name="MiR_surface"/>
             <!-- IMU -->
-                <joint name="MiR__base_to_imu_joint" type="fixed">
+                <joint name="MiR__base_to_imu_joint_fixed" type="fixed">
                     <parent link="MiR_base_link" />
                     <child link="MiR_imu_link" />
@@ -166,5 +168,5 @@
                     TF has imu_link, but the imu_data topic is published in the imu_frame
                     frame. -->
-                    <joint name="MiR__imu_link_to_imu_frame_joint" type="fixed">
+                    <joint name="MiR__imu_link_to_imu_frame_joint_fixed" type="fixed">
                         <parent link="MiR_imu_link" />
                         <child link="MiR_imu_frame" />
@@ -191,5 +193,5 @@
                     </xacro:box_inertial>
                 </link>
-                <joint name="MiR__base_to_front_laser_joint" type="fixed">
+                <joint name="MiR__base_to_front_laser_joint_fixed" type="fixed">
                     <parent link="MiR_base_link" />
                     <child link="MiR_front_laser_link" />
@@ -214,5 +216,5 @@
                     </xacro:box_inertial>
                 </link>
-                <joint name="Mir__base_to_back_laser_joint" type="fixed">
+                <joint name="Mir__base_to_back_laser_joint_fixed" type="fixed">
                     <parent link="MiR_base_link" />
                     <child link="MiR_back_laser_link" />
@@ -221,5 +223,5 @@
             <!-- Ultrasound sensors -->
                 <link name="MiR_right_us_frame" />
-                <joint name="MiR__base_to_right_us_joint" type="fixed">
+                <joint name="MiR__base_to_right_us_joint_fixed" type="fixed">
                     <parent link="MiR_base_link" />
                     <child link="MiR_right_us_frame" />
@@ -227,5 +229,5 @@
                 </joint>
                 <link name="MiR_left_us_frame" />
-                <joint name="MiR__base_to_left_us_joint" type="fixed">
+                <joint name="MiR__base_to_left_us_joint_fixed" type="fixed">
                     <parent link="MiR_base_link" />
                     <child link="MiR_left_us_frame" />

File: urdf/mir100/mir100_mobile_robot.xacro (robot description, xacro)
@@ -23,5 +23,6 @@
             <xacro:set_wheel_friction link="MiR_br_caster_wheel_link" friction="1"/>
             <xacro:p3d_base_controller/>
-            <xacro:MiR100_controller/>
+            <xacro:MiR_controller_plugin_gazebo left_wheel_joint="MiR__base_left_wheel_joint" right_wheel_joint="MiR__base_right_wheel_joint" wheel_separation="${wheel_separation}" wheel_radius="${wheel_radius}"/>
+            <!-- <xacro:MiR100_controller/> -->
             <xacro:MiR100_gazebo/>
         <!-- ############## Gazebo ####################### -->

File: urdf/mobile_manipulator.xacro (robot description, xacro)
@@ -30,5 +30,5 @@
             <xacro:set_wheel_friction link="MiR_br_caster_wheel_link" friction="1"/>
             <xacro:p3d_base_controller/>
-            <!-- <xacro:UR10_controller/> is already Included. BH282_controller is duplication of UR10_controller -->
+            <xacro:MiR_controller_plugin_gazebo left_wheel_joint="MiR__base_left_wheel_joint" right_wheel_joint="MiR__base_right_wheel_joint" wheel_separation="${wheel_separation}" wheel_radius="${wheel_radius}"/>
             <!-- <xacro:MiR100_controller/> -->
             <xacro:MiR100_gazebo/>

File: urdf/ur10/ur10.urdf.xacro (robot description, xacro)
@@ -50,5 +50,5 @@
     <!-- ############################################### -->
         <xacro:macro name="UR10_arm" params="parent">
-            <joint name="UR10_base_joint" type="fixed">
+            <joint name="UR10_base_joint_fixed" type="fixed">
                 <origin xyz="0.15 0.0 0.352" rpy="0.0 0.0 0.0" />
                 <parent link="${parent}"/>
@@ -247,5 +247,5 @@
                 </xacro:cylinder_inertial>
             </link>
-            <joint name="UR10__wrist_3_to_end_effector_fixed_joint" type="fixed">
+            <joint name="UR10__wrist_3_to_end_effector_joint_fixed" type="fixed">
                 <parent link="UR10_wrist_3_link" />
                 <child link = "UR10_end_effector_link" />
