Commit message: Mobile Manipulator is working fine. The Controller for the hand switched to effort controller and stopped_velocity_tolerance ncreased from 0.0

File: urdf/bh282/bh282.transmission.xacro (robot description, xacro)
@@ -5,5 +5,5 @@
         <xacro:macro name="BH282_joint_transmission"
                         params="joint
-                                hw_interface:=hardware_interface/PositionJointInterface
+                                hw_interface:=hardware_interface/EffortJointInterface
                                 tm_type:=transmission_interface/SimpleTransmission">
             <transmission name="BH282__${joint}_trans">

File: urdf/bh282/bh282.urdf.xacro (robot description, xacro)
@@ -3,9 +3,10 @@
     <!-- ################# Properties ################ -->
     <!-- ############################################# -->
-        <xacro:property name="BH282_joint_damping" value="100.0" />
-        <xacro:property name="BH282_joint_friction" value="1.0" />
+        <xacro:property name="BH282_joint_damping" value="0.7" />
+        <xacro:property name="BH282_joint_friction" value="0.0" />
         <xacro:property name="BH282_joint_effort_limit" value="30.0" />
         <xacro:property name="BH282_joint_velocity_limit" value="2.0" />
         <xacro:property name="BH282_mechanical_reduction" value="1.0" />
+        <xacro:property name="BH282_friction_coefficient" value="100.0" />
     <!-- ############################################# -->
     <!-- ################# Properties ################ -->
@@ -16,6 +17,6 @@
                 <!-- To Attach the Gripper to the Arm -->
                 <!-- Change This if you would like to run the gripper stand-alone -->
-                <!-- <origin xyz="0 0 0" rpy="0 ${0.5 * pi} 0" /> -->
-                <origin xyz="0 0 0" rpy="0 0 0" />
+                <origin xyz="0 0 0" rpy="0 ${0.5 * pi} 0" />
+                <!-- <origin xyz="0 0 0" rpy="0 0 0" /> -->
                 <parent link="${parent}"/>
                 <child link="BH282_base_link"/>
@@ -39,5 +40,5 @@
                         <mesh filename="package://mobile_manipulator/mesh/barrett/palm_282.dae"/>
                     </geometry>
-                    <contact_coefficients kd="1.0" kp="1000.0" mu="0"/>
+                    <contact_coefficients kd="1.0" kp="1000.0" mu="${BH282_friction_coefficient}"/>
                 </collision>
             </link>
